Commit message: Spawn two robots Rick & Morty, publish to their own channels

File: xacro/barista_robot_model.urdf.xacro (robot description, xacro)
@@ -2,4 +2,5 @@
 <robot xmlns:xacro="http://www.ros.org/wiki/xacro" name="barista_robot">
   <!-- Conditional Argument -->
+  <xacro:property name="robot_name" value="$(arg robot_name)"/>
   <xacro:arg name="include_laser" default="true"/>
   <!-- Macro Includes -->
@@ -10,7 +11,7 @@
   <xacro:include filename="$(find barista_robot_description)/xacro/laser_scanner.xacro"/>
   <!-- Materials -->
-  <material name="blue"><color rgba="0.0 0.0 1.0 1"/></material>
-  <material name="black"><color rgba="0.0 0.0 0.0 1"/></material>
-  <material name="grey"><color rgba="0.75 0.75 0.75 1"/></material>
+  <material name="$(arg robot_name)_blue"><color rgba="0.0 0.0 1.0 1"/></material>
+  <material name="$(arg robot_name)_black"><color rgba="0.0 0.0 0.0 1"/></material>
+  <material name="$(arg robot_name)_grey"><color rgba="0.75 0.75 0.75 1"/></material>
   <!-- Base Link & Main Body -->
   <link name="base_link"/>
@@ -18,5 +19,5 @@
     <visual>
       <geometry><cylinder radius="0.178" length="0.155"/></geometry>
-      <material name="blue"/>
+      <material name="$(arg robot_name)_blue"/>
     </visual>
     <collision>
@@ -54,5 +55,5 @@
   <gazebo>
     <plugin filename="gz-sim-joint-state-publisher-system" name="gz::sim::systems::JointStatePublisher">
-      <topic>/joint_states</topic>
+      <topic>${robot_name}/joint_states</topic>
       <update_rate>30</update_rate>
       <joint_name>joint_drive_wheel_left</joint_name>
@@ -72,17 +73,12 @@
       <wheel_separation>0.256</wheel_separation>
       <wheel_radius>0.0352</wheel_radius>
-      <topic>cmd_vel</topic>
+      <topic>${robot_name}/cmd_vel</topic>
       <publish_odom>true</publish_odom>
       <publish_odom_tf>true</publish_odom_tf>
       <publish_wheel_tf>true</publish_wheel_tf>
-      <odom_topic>odom</odom_topic>
+      <odom_topic>${robot_name}/odom</odom_topic>
       <tf_topic>tf</tf_topic>
-      <frame_id>odom</frame_id>
-      <child_frame_id>base_link</child_frame_id>
-    </plugin>
-  </gazebo>
-  <gazebo>
-    <plugin filename="gz-sim-sensors-system" name="gz::sim::systems::Sensors">
-      <render_engine>ogre2</render_engine>
+      <frame_id>${robot_name}/odom</frame_id>
+      <child_frame_id>${robot_name}/base_link</child_frame_id>
     </plugin>
   </gazebo>

File: xacro/caster_wheel.xacro (robot description, xacro)
@@ -9,5 +9,5 @@
                 <cylinder length="0.005" radius="0.0352"/>
             </geometry>
-            <material name="black"/>
+            <material name="$(arg robot_name)_black"/>
         </visual>
         <collision>
@@ -38,5 +38,5 @@
                 <cylinder length="0.005" radius="0.0352"/>
             </geometry>
-            <material name="black"/>
+            <material name="$(arg robot_name)_black"/>
         </visual>
         <collision>
@@ -67,5 +67,5 @@
                 <sphere radius="0.0352"/>
             </geometry>
-            <material name="black"/>
+            <material name="$(arg robot_name)_black"/>
         </visual>
         <collision>

File: xacro/cup_holder_tray.xacro (robot description, xacro)
@@ -8,5 +8,5 @@
       <visual>
         <geometry><cylinder radius="${tray_radius}" length="${tray_length}"/></geometry>
-        <material name="blue"/>
+        <material name="$(arg robot_name)_blue"/>
       </visual>
       <collision>

File: xacro/drive_wheel.xacro (robot description, xacro)
@@ -11,5 +11,5 @@
           <cylinder radius="${wheel_radius}" length="${wheel_width}"/>
         </geometry>
-        <material name="black"/>
+        <material name="$(arg robot_name)_black"/>
       </visual>
       <collision>

File: xacro/laser_scanner.xacro (robot description, xacro)
@@ -1,5 +1,5 @@
 <?xml version="1.0"?>
 <robot xmlns:xacro="http://www.ros.org/wiki/xacro">
-  <xacro:macro name="laser_scanner" params="parent origin_xyz">
+<xacro:macro name="laser_scanner" params="parent origin_xyz">
     <link name="laser_scan_link">
         <visual>
@@ -36,9 +36,9 @@
       <sensor type="gpu_lidar" name="gpu_lidar">
         <pose relative_to='laser_scan_frame'>0 0 0 0 0 0</pose>
-        <gz_frame_id>laser_scan_frame</gz_frame_id>
+        <gz_frame_id>${robot_name}/laser_scan_frame</gz_frame_id>
         <always_on>1</always_on>
         <visualize>true</visualize>
         <update_rate>30</update_rate>
-        <topic>scan</topic>
+        <topic>${robot_name}/scan</topic>
         <ray>
           <scan>
@@ -58,3 +58,4 @@
       </sensor>
     </gazebo>
+</xacro:macro>
 </robot>

File: xacro/standoff_rod.xacro (robot description, xacro)
@@ -5,5 +5,5 @@
       <visual>
         <geometry><cylinder radius="${radius}" length="${length}"/></geometry>
-        <material name="grey"/>
+        <material name="$(arg robot_name)_grey"/>
       </visual>
       <collision>

Commit message: Fix Rick colour to Red and Morty to Blue

File: xacro/barista_robot_model.urdf.xacro (robot description, xacro)
@@ -3,4 +3,5 @@
   <!-- Conditional Argument -->
   <xacro:property name="robot_name" value="$(arg robot_name)"/>
+  <xacro:arg name="robot_color" default="blue"/>
   <xacro:arg name="include_laser" default="true"/>
   <!-- Macro Includes -->
@@ -12,4 +13,5 @@
   <!-- Materials -->
   <material name="$(arg robot_name)_blue"><color rgba="0.0 0.0 1.0 1"/></material>
+  <material name="$(arg robot_name)_red"><color rgba="1.0 0.0 0.0 1"/></material>
   <material name="$(arg robot_name)_black"><color rgba="0.0 0.0 0.0 1"/></material>
   <material name="$(arg robot_name)_grey"><color rgba="0.75 0.75 0.75 1"/></material>
@@ -19,5 +21,5 @@
     <visual>
       <geometry><cylinder radius="0.178" length="0.155"/></geometry>
-      <material name="$(arg robot_name)_blue"/>
+      <material name="$(arg robot_name)_$(arg robot_color)"/>
     </visual>
     <collision>

File: xacro/cup_holder_tray.xacro (robot description, xacro)
@@ -8,5 +8,5 @@
       <visual>
         <geometry><cylinder radius="${tray_radius}" length="${tray_length}"/></geometry>
-        <material name="$(arg robot_name)_blue"/>
+        <material name="$(arg robot_name)_$(arg robot_color)"/>
       </visual>
       <collision>
