Commit message: fix robot body and drive wheel dimensions/placement + add collision and inertial info

File: urdf/barista_robot_model.urdf (robot description, URDF)
Before this commit: robot barista_robot, 15 links, 14 joints
Links:
- link back_pitch_link: mass None -> 0.001; geometry collision sphere radius=0.01; visual sphere radius=0.01
- link back_roll_link: mass None -> 0.001; geometry collision cylinder length=0.001 radius=0.0045000000000000005; visual cylinder length=0.001 radius=0.0045000000000000005
- link back_yaw_link: mass None -> 0.001; geometry collision cylinder length=0.001 radius=0.0045000000000000005; visual cylinder length=0.001 radius=0.0045000000000000005
- link cup_holder_tray: mass None -> 0.25; geometry collision cylinder length=.09 radius=0.16; visual cylinder length=.09 radius=0.16
- link drive_wheel_left: mass None -> 0.05; geometry collision cylinder length=0.0206 radius=0.0352; visual cylinder length=0.0206 radius=0.0352
- link drive_wheel_right: mass None -> 0.05; geometry collision cylinder length=0.0206 radius=0.0352; visual cylinder length=0.0206 radius=0.0352
- link front_pitch_link: mass None -> 0.001; geometry collision sphere radius=0.01; visual sphere radius=0.01
- link front_roll_link: mass None -> 0.001; geometry collision cylinder length=0.001 radius=0.0045000000000000005; visual cylinder length=0.001 radius=0.0045000000000000005
- link front_yaw_link: mass None -> 0.001; geometry collision cylinder length=0.001 radius=0.0045000000000000005; visual cylinder length=0.001 radius=0.0045000000000000005
- link main_body: mass None -> 0.5; geometry collision cylinder length=0.155 radius=0.178; visual cylinder length=0.155 radius=0.178
- link standoff_rod_1: mass None -> 0.075; geometry collision cylinder length=.220 radius=.01; visual cylinder length=.220 radius=.01
- link standoff_rod_2: mass None -> 0.075; geometry collision cylinder length=.220 radius=.01; visual cylinder length=.220 radius=.01
- link standoff_rod_3: mass None -> 0.075; geometry collision cylinder length=.220 radius=.01; visual cylinder length=.220 radius=.01
- link standoff_rod_4: mass None -> 0.075; geometry collision cylinder length=.220 radius=.01; visual cylinder length=.220 radius=.01
Joints:
- joint joint_drive_wheel_left: origin xyz=0 0.05 -0.025 rpy=0 0 0 -> xyz=0 0.11 -0.0775 rpy=0 0 0
- joint joint_drive_wheel_right: origin xyz=0 -0.05 -0.025 rpy=0 0 0 -> xyz=0 -0.11 -0.0775 rpy=0 0 0
- joint main_link_to_rod1_joint: origin xyz=0.10 0.06 0.1875 rpy=0 0 0 -> xyz=0.06 0.10 0.1875 rpy=0 0 0
- joint main_link_to_rod2_joint: origin xyz=-0.10 0.06 0.1875 rpy=0 0 0 -> xyz=-0.06 0.10 0.1875 rpy=0 0 0
- joint main_link_to_rod3_joint: origin xyz=-0.10 -0.06 0.1875 rpy=0 0 0 -> xyz=-0.06 -0.10 0.1875 rpy=0 0 0
- joint main_link_to_rod4_joint: origin xyz=0.10 -0.06 0.1875 rpy=0 0 0 -> xyz=0.06 -0.10 0.1875 rpy=0 0 0

Commit message: Adjust drive wheel z axis placement tomatch small caster wheel

File: urdf/barista_robot_model.urdf (robot description, URDF)
Before this commit: robot barista_robot, 15 links, 14 joints
Joints:
- joint back_yaw_joint: origin xyz=-0.04 0 -0.05 rpy=0 0 0 -> xyz=-0.11 0 -0.0775 rpy=0 0 0
- joint front_yaw_joint: origin xyz=0.04 0 -0.05 rpy=0 0 0 -> xyz=0.11 0 -0.0775 rpy=0 0 0
- joint joint_drive_wheel_left: origin xyz=0 0.11 -0.0775 rpy=0 0 0 -> xyz=0 0.11 -0.0523 rpy=0 0 0
- joint joint_drive_wheel_right: origin xyz=0 -0.11 -0.0775 rpy=0 0 0 -> xyz=0 -0.11 -0.0523 rpy=0 0 0

Commit message: Attempting to make laser_scan work and initialize gazebo sim

File: urdf/barista_robot_model.urdf (robot description, URDF)
Before this commit: robot barista_robot, 15 links, 14 joints
Links:
- added link laser_scan_frame
- added link laser_scan_link, mass 0.01; collision box size=0.02 0.02 0.02; visual box size=0.02 0.02 0.02
- added link laser_scan_model_link, mass 0.01; collision cylinder length=0.0408 radius=0.037493; visual mesh filename=package://barista_robot_description/meshes/slamtec_rplidar_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 scale=1.0 1.0 1.0
Joints:
- added joint laser_scan_frame_joint: type fixed, parent laser_scan_link, child laser_scan_frame, origin xyz=0 0 0.03 rpy=0 0 0, axis 0 0 0
- added joint laser_scan_link_joint: type continuous, parent main_body, child laser_scan_link, origin xyz=0.0 0.0 0.05 rpy=0 0 0, axis 0 0 1, limit lower=-0.1 upper=0.0 effort=20.0 velocity=2.0
- added joint laser_scan_model_link_joint: type continuous, parent laser_scan_link, child laser_scan_model_link, origin xyz=0.11 0.0 0.0275 rpy=0 0 0, axis 0 0 1, limit effort=10.0 velocity=2.0

Commit message: Fix laser_scan_link_joint and laser_scan_model_link_joint, ros2_control_config and config files to ensure launch file runs

File: urdf/barista_robot_model.urdf (robot description, URDF)
Before this commit: robot barista_robot, 18 links, 17 joints
Joints:
- joint laser_scan_link_joint: axis 0 0 1 -> (none); limit lower=-0.1 upper=0.0 effort=20.0 velocity=2.0 -> (none); origin xyz=0.0 0.0 0.05 rpy=0 0 0 -> xyz=0.0 0.0 0.0775 rpy=0 0 0; type continuous -> fixed
- joint laser_scan_model_link_joint: origin xyz=0.11 0.0 0.0275 rpy=0 0 0 -> xyz=0.11 0.0 0.0 rpy=0 0 0

Commit message: fix laser scanner position to be offset, task 1 complete

File: urdf/barista_robot_model.urdf (robot description, URDF)
Before this commit: robot barista_robot, 18 links, 17 joints
Joints:
- joint laser_scan_link_joint: origin xyz=0.0 0.0 0.0775 rpy=0 0 0 -> xyz=0.11 0.0 0.0775 rpy=0 0 0
- joint laser_scan_model_link_joint: origin xyz=0.11 0.0 0.0 rpy=0 0 0 -> xyz=0.0 0.0 0.0 rpy=0 0 0

Commit message: Fixed mistakes from URDF Checkpoint submission, referred to solution packet

File: urdf/barista_robot_model.urdf (robot description, URDF)
Before this commit: robot barista_robot, 18 links, 17 joints
Links:
- removed link laser_scan_model_link
- link back_pitch_link: mass 0.001 -> 0.01; geometry collision sphere radius=0.0352; visual sphere radius=0.0352
- link back_roll_link: mass 0.001 -> 0.01; geometry collision cylinder length=0.005 radius=0.0352; visual cylinder length=0.005 radius=0.0352
- link back_yaw_link: mass 0.001 -> 0.01; geometry collision cylinder length=0.005 radius=0.0352; visual cylinder length=0.005 radius=0.0352
- link cup_holder_tray: mass 0.25 -> 0.05
- link drive_wheel_left: mass 0.05 -> 0.01
- link drive_wheel_right: mass 0.05 -> 0.01
- link front_pitch_link: mass 0.001 -> 0.01; geometry collision sphere radius=0.0352; visual sphere radius=0.0352
- link front_roll_link: mass 0.001 -> 0.01; geometry collision cylinder length=0.005 radius=0.0352; visual cylinder length=0.005 radius=0.0352
- link front_yaw_link: mass 0.001 -> 0.01; geometry collision cylinder length=0.005 radius=0.0352; visual cylinder length=0.005 radius=0.0352
- link laser_scan_link: geometry collision box size=0.074986 0.074935 0.0408; visual mesh filename=package://barista_robot_description/meshes/slamtec_rplidar_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 scale=1.0 1.0 1.0
- link main_body: mass 0.5 -> 0.2
- link standoff_rod_1: mass 0.075 -> 0.02
- link standoff_rod_2: mass 0.075 -> 0.02
- link standoff_rod_3: mass 0.075 -> 0.02
- link standoff_rod_4: mass 0.075 -> 0.02
Joints:
- removed joint laser_scan_model_link_joint
- joint back_yaw_joint: origin xyz=-0.11 0 -0.0775 rpy=0 0 0 -> xyz=-0.12 0 -0.0775 rpy=0 0 0
- joint front_yaw_joint: origin xyz=0.11 0 -0.0775 rpy=0 0 0 -> xyz=0.12 0 -0.0775 rpy=0 0 0
- joint joint_drive_wheel_left: origin xyz=0 0.11 -0.0523 rpy=0 0 0 -> xyz=0 0.128 -0.0775 rpy=0 0 0
- joint joint_drive_wheel_right: origin xyz=0 -0.11 -0.0523 rpy=0 0 0 -> xyz=0 -0.128 -0.0775 rpy=0 0 0
- joint laser_scan_link_joint: origin xyz=0.0 0.0 0.0775 rpy=0 0 0 -> xyz=0.1 0.0 0.0775 rpy=0 0 0
- joint main_link_to_rod1_joint: origin xyz=0.06 0.10 0.1875 rpy=0 0 0 -> xyz=0.05 0.12 0.1875 rpy=0 0 0
- joint main_link_to_rod2_joint: origin xyz=-0.06 0.10 0.1875 rpy=0 0 0 -> xyz=-0.05 0.12 0.1875 rpy=0 0 0
- joint main_link_to_rod3_joint: origin xyz=-0.06 -0.10 0.1875 rpy=0 0 0 -> xyz=-0.05 -0.12 0.1875 rpy=0 0 0
- joint main_link_to_rod4_joint: origin xyz=0.06 -0.10 0.1875 rpy=0 0 0 -> xyz=0.05 -0.12 0.1875 rpy=0 0 0

File: xacro/barista_robot_model.urdf.xacro (robot description, xacro)
@@ -24,7 +24,7 @@
     </collision>
     <inertial>
-      <mass value="0.5"/>
-      <origin rpy="0 0 0" xyz="0 0 0"/>
-      <inertia ixx="0.004962" ixy="0" ixz="0" iyy="0.004962" iyz="0" izz="0.007921"/>
+        <mass value="0.2"/>
+        <origin rpy="0 0 0" xyz="0 0 0"/>
+        <inertia ixx="0.0019846" ixy="0" ixz="0" iyy="0.0019846" iyz="0" izz="0.0031684"/>
     </inertial>
   </link>
@@ -35,19 +35,19 @@
   </joint>
   <!-- Drive Wheels -->
-  <xacro:drive_wheel location="left" parent="main_body" origin_xyz="0 0.11 -0.0523"/>
-  <xacro:drive_wheel location="right" parent="main_body" origin_xyz="0 -0.11 -0.0523"/>
+  <xacro:drive_wheel location="left" parent="main_body" origin_xyz="0 0.128 -0.0775"/>
+  <xacro:drive_wheel location="right" parent="main_body" origin_xyz="0 -0.128 -0.0775"/>
   <!-- Casters -->
-  <xacro:caster_wheel location="front" parent="main_body" origin_xyz="0.11 0 -0.0775"/>
-  <xacro:caster_wheel location="back" parent="main_body" origin_xyz="-0.11 0 -0.0775"/>
+  <xacro:caster_wheel location="front" parent="main_body" origin_xyz="0.12 0 -0.0775"/>
+  <xacro:caster_wheel location="back" parent="main_body" origin_xyz="-0.12 0 -0.0775"/>
   <!-- Standoff Rods -->
-  <xacro:standoff_rod prefix="1" parent="main_body" origin_xyz="0.06 0.10 0.1875"/>
-  <xacro:standoff_rod prefix="2" parent="main_body" origin_xyz="-0.06 0.10 0.1875"/>
-  <xacro:standoff_rod prefix="3" parent="main_body" origin_xyz="-0.06 -0.10 0.1875"/>
-  <xacro:standoff_rod prefix="4" parent="main_body" origin_xyz="0.06 -0.10 0.1875"/>
+  <xacro:standoff_rod prefix="1" parent="main_body" origin_xyz="0.05 0.12 0.1875"/>
+  <xacro:standoff_rod prefix="2" parent="main_body" origin_xyz="-0.05 0.12 0.1875"/>
+  <xacro:standoff_rod prefix="3" parent="main_body" origin_xyz="-0.05 -0.12 0.1875"/>
+  <xacro:standoff_rod prefix="4" parent="main_body" origin_xyz="0.05 -0.12 0.1875"/>
   <!-- Cup Holder Tray -->
   <xacro:cup_holder_tray parent="main_body" origin_xyz="0 0 0.3425"/>
   <!-- Conditional Laser Scanner -->
   <xacro:if value="$(arg include_laser)">
-    <xacro:laser_scanner parent="main_body" origin_xyz="0.11 0.0 0.0775"/>
+    <xacro:laser_scanner parent="main_body" origin_xyz="0.1 0.0 0.0775"/>
   </xacro:if>
   <!-- Gazebo Core Plugins -->
@@ -70,5 +70,5 @@
       <left_joint>joint_drive_wheel_left</left_joint>
       <right_joint>joint_drive_wheel_right</right_joint>
-      <wheel_separation>0.22</wheel_separation>
+      <wheel_separation>0.256</wheel_separation>
       <wheel_radius>0.0352</wheel_radius>
       <topic>cmd_vel</topic>

File: xacro/caster_wheel.xacro (robot description, xacro)
@@ -4,18 +4,22 @@
     <!-- Yaw Link -->
     <link name="${location}_yaw_link">
-      <visual>
-        <origin rpy="0 1.5707 1.5707" xyz="0 0 0"/>
-        <geometry><cylinder length="0.001" radius="0.0045"/></geometry>
-        <material name="black"/>
-      </visual>
-      <collision>
-        <origin rpy="0 1.5707 1.5707" xyz="0 0 0"/>
-        <geometry><cylinder length="0.001" radius="0.0045"/></geometry>
-      </collision>
-      <inertial>
-        <origin rpy="0 1.5707 1.5707" xyz="0 0 0"/>
-        <mass value="0.001"/>
-        <inertia ixx="5.145e-09" ixy="0" ixz="0" iyy="5.145e-09" iyz="0" izz="1.0125e-08"/>
-      </inertial>
+        <visual>
+            <origin rpy="0 1.5707 1.5707" xyz="0 0 0"/>
+            <geometry>
+                <cylinder length="0.005" radius="0.0352"/>
+            </geometry>
+            <material name="black"/>
+        </visual>
+        <collision>
+            <origin rpy="0 1.5707 1.5707" xyz="0 0 0"/>
+            <geometry>
+                <cylinder length="0.005" radius="0.0352"/>
+            </geometry>
+        </collision>
+        <inertial>
+            <mass value="0.01"/>
+            <origin rpy="0 0 0" xyz="0 0 0"/>
+            <inertia ixx="0.0000031184" ixy="0" ixz="0" iyy="0.0000031184" iyz="0" izz="0.000006195"/>
+        </inertial>
     </link>
     <joint name="${location}_yaw_joint" type="continuous">
@@ -29,18 +33,22 @@
     <!-- Roll Link -->
     <link name="${location}_roll_link">
-      <visual>
-        <origin rpy="0 1.5707 1.5707" xyz="0 0 0"/>
-        <geometry><cylinder length="0.001" radius="0.0045"/></geometry>
-        <material name="black"/>
-      </visual>
-      <collision>
-        <origin rpy="0 1.5707 1.5707" xyz="0 0 0"/>
-        <geometry><cylinder length="0.001" radius="0.0045"/></geometry>
-      </collision>
-      <inertial>
-        <origin rpy="0 1.5707 1.5707" xyz="0 0 0"/>
-        <mass value="0.001"/>
-        <inertia ixx="5.145e-09" ixy="0" ixz="0" iyy="5.145e-09" iyz="0" izz="1.0125e-08"/>
-      </inertial>
+        <visual>
+            <origin rpy="0 1.5707 1.5707" xyz="0 0 0"/>
+            <geometry>
+                <cylinder length="0.005" radius="0.0352"/>
+            </geometry>
+            <material name="black"/>
+        </visual>
+        <collision>
+            <origin rpy="0 1.5707 1.5707" xyz="0 0 0"/>
+            <geometry>
+                <cylinder length="0.005" radius="0.0352"/>
+            </geometry>
+        </collision>
+        <inertial>
+            <mass value="0.01"/>
+            <origin rpy="0 0 0" xyz="0 0 0"/>
+            <inertia ixx="0.0000031184" ixy="0" ixz="0" iyy="0.0000031184" iyz="0" izz="0.000006195"/>
+        </inertial>
     </link>
     <joint name="${location}_roll_joint" type="continuous">
@@ -54,24 +62,28 @@
     <!-- Pitch Link (Sphere Contact) -->
     <link name="${location}_pitch_link">
-      <visual>
-        <origin rpy="0 1.5707 1.5707" xyz="0 0 0"/>
-        <geometry><sphere radius="0.01"/></geometry>
-        <material name="black"/>
-      </visual>
-      <collision>
-        <origin rpy="0 1.5707 1.5707" xyz="0 0 0"/>
-        <geometry><sphere radius="0.01"/></geometry>
-      </collision>
-      <inertial>
-        <origin rpy="0 1.5707 1.5707" xyz="0 0 0"/>
-        <mass value="0.001"/>
-        <inertia ixx="4e-08" ixy="0" ixz="0" iyy="4e-08" iyz="0" izz="4e-08"/>
-      </inertial>
+        <visual>
+            <origin rpy="0 1.5707 1.5707" xyz="0 0 0"/>
+            <geometry>
+                <sphere radius="0.0352"/>
+            </geometry>
+            <material name="black"/>
+        </visual>
+        <collision>
+            <origin rpy="0 1.5707 1.5707" xyz="0 0 0"/>
+            <geometry>
+                <sphere radius="0.0352"/>
+            </geometry>
+        </collision>
+        <inertial>
+            <mass value="0.01"/>
+            <origin rpy="0 0 0" xyz="0 0 0"/>
+            <inertia ixx="0.00000826" ixy="0" ixz="0" iyy="00.00000826" iyz="0" izz="0.00000826"/>
+        </inertial>
     </link>
     <gazebo reference="${location}_pitch_link">
       <collision>
         <surface>
-          <friction><ode><mu>0.5</mu><mu2>0.5</mu2></ode></friction>
-          <contact><ode><kp>10000000.0</kp><kd>10000000.0</kd></ode></contact>
+          <friction><ode><mu>0.1</mu><mu2>0.1</mu2></ode></friction>
+          <contact><ode><kp>1000000000000000000000000000.0</kp><kd>1000000000000000000000000000.0</kd></ode></contact>
         </surface>
       </collision>

File: xacro/cup_holder_tray.xacro (robot description, xacro)
@@ -14,7 +14,7 @@
       </collision>
       <inertial>
-        <mass value="0.25"/>
+        <mass value="0.05"/>
         <origin rpy="0 0 0" xyz="0 0 0"/>
-        <inertia ixx="0.0017688" ixy="0" ixz="0" iyy="0.0017688" iyz="0" izz="0.0032"/>
+        <inertia ixx="0.00035375" ixy="0" ixz="0" iyy="0.00035375" iyz="0" izz="0.00064"/>
       </inertial>
     </link>

File: xacro/drive_wheel.xacro (robot description, xacro)
@@ -20,7 +20,7 @@
       </collision>
       <inertial>
-        <mass value="0.05"/>
-        <origin rpy="0 1.5707 1.5707" xyz="0 0 0"/>
-        <inertia ixx="0.000017256" ixy="0" ixz="0" iyy="0.000017256" iyz="0" izz="0.000030976"/>
+        <mass value="0.01"/>
+        <origin rpy="0 0 0" xyz="0 0 0"/>
+        <inertia ixx="0.000003451" ixy="0" ixz="0" iyy="0.000003451" iyz="0" izz="0.000006195"/>
       </inertial>
     </link>
@@ -36,6 +36,6 @@
           <contact>
             <ode>
-              <kp>10000000.0</kp>
-              <kd>10000000.0</kd>
+              <kp>1000000000000000000000000000.0</kp>
+              <kd>1000000000000000000000000000.0</kd>
             </ode>
           </contact>

File: xacro/laser_scanner.xacro (robot description, xacro)
@@ -3,17 +3,21 @@
   <xacro:macro name="laser_scanner" params="parent origin_xyz">
     <link name="laser_scan_link">
-      <visual>
-        <origin rpy="0 0 0" xyz="0 0 0"/>
-        <geometry><box size="0.02 0.02 0.02"/></geometry>
-      </visual>
-      <collision>
-        <origin rpy="0 0 0" xyz="0 0 0.0204"/>
-        <geometry><box size="0.02 0.02 0.02"/></geometry>
-      </collision>
-      <inertial>
-        <mass value="0.01"/>
-        <origin rpy="0 0 0" xyz="0 0 0.01"/>
-        <inertia ixx="6.0665e-06" ixy="0" ixz="0" iyy="6.0729e-06" iyz="0" izz="9.3651e-06"/>
-      </inertial>
+        <visual>
+            <origin rpy="0 0 0" xyz="0 0 0"/>
+            <geometry>
+                <mesh filename="package://barista_robot_description/meshes/slamtec_rplidar_s1.dae" scale="1.0 1.0 1.0"/>
+            </geometry>
+        </visual>
+        <collision>
+            <origin rpy="0 0 0" xyz="0 0 0.0204"/>
+            <geometry>
+                <box size="0.074986 0.074935 0.0408"/>
+            </geometry>
+        </collision>
+        <inertial>
+            <mass value="0.01"/>
+            <origin rpy="0 0 0" xyz="0 0 0.0204"/>
+            <inertia ixx="6.066578520833334e-06" ixy="0" ixz="0" iyy="6.072950163333333e-06" iyz="0" izz="9.365128684166666e-06"/>
+        </inertial>
     </link>
     <joint name="laser_scan_link_joint" type="fixed">
@@ -28,30 +32,4 @@
       <child link="laser_scan_frame"/>
     </joint>
-    <!-- Mesh Visual Model -->
-    <link name="laser_scan_model_link">
-      <visual>
-        <origin rpy="0 0 0" xyz="0 0 0"/>
-        <geometry>
-          <mesh filename="package://barista_robot_description/meshes/slamtec_rplidar_s1.dae" scale="1.0 1.0 1.0"/>
-        </geometry>
-      </visual>
-      <collision>
-        <origin rpy="0 0 0" xyz="0 0 0.0204"/>
-        <geometry><cylinder length="0.0408" radius="0.037493"/></geometry>
-      </collision>
-      <inertial>
-        <mass value="0.01"/>
-        <origin rpy="0 0 0" xyz="0 0 0.0204"/>
-        <inertia ixx="6.0665e-06" ixy="0" ixz="0" iyy="6.0729e-06" iyz="0" izz="9.3651e-06"/>
-      </inertial>
-    </link>
-    <joint name="laser_scan_model_link_joint" type="continuous">
-      <origin rpy="0 0 0" xyz="0.0 0.0 0.0"/>
-      <parent link="laser_scan_link"/>
-      <child link="laser_scan_model_link"/>
-      <axis xyz="0 0 1"/>
-      <limit effort="10.0" velocity="2.0"/>
-      <dynamics friction="0.01"/>
-    </joint>
     <!-- Laser Scanner Sensor Plugin -->
     <gazebo reference="laser_scan_frame">
@@ -61,5 +39,5 @@
         <always_on>1</always_on>
         <visualize>true</visualize>
-        <update_rate>100</update_rate>
+        <update_rate>30</update_rate>
         <topic>scan</topic>
         <ray>
@@ -80,24 +58,3 @@
       </sensor>
     </gazebo>
-    <ros2_control name="GazeboSimSystem" type="system">
-      <hardware>
-        <plugin>gz_ros2_control/GazeboSimSystem</plugin>
-      </hardware>
-      <joint name="laser_scan_model_link_joint">
-        <command_interface name="velocity">
-          <param name="min">0.0</param>
-          <param name="max">2.0</param>
-        </command_interface>
-        <state_interface name="position"/>
-        <state_interface name="velocity"/>
-        <state_interface name="effort"/>
-      </joint>
-    </ros2_control>
-    <!-- Gazebo ROS 2 Control Plugin -->
-    <gazebo>
-      <plugin filename="gz_ros2_control-system" name="gz_ros2_control::GazeboSimROS2ControlPlugin">
-        <parameters>$(find barista_robot_description)/config/controller_position_velocity.yaml</parameters>
-      </plugin>
-    </gazebo>
-  </xacro:macro>
 </robot>

File: xacro/standoff_rod.xacro (robot description, xacro)
@@ -11,7 +11,7 @@
       </collision>
       <inertial>
-        <mass value="0.075"/>
+        <mass value="0.02"/>
         <origin rpy="0 0 0" xyz="0 0 0"/>
-        <inertia ixx="0.0003044" ixy="0" ixz="0" iyy="0.0003044" iyz="0" izz="0.00000375"/>
+        <inertia ixx="0.00008117" ixy="0" ixz="0" iyy="0.00008117" iyz="0" izz="0.000001"/>
       </inertial>
     </link>

Commit message: Fix physics-related URDF file issue causing Morty to get stuck in Gazebo

File: urdf/barista_robot_model.urdf (robot description, URDF)
Before this commit: robot barista_robot, 17 links, 16 joints
Links:
- link back_roll_link: geometry visual cylinder length=0.005 radius=0.0352
- link back_yaw_link: geometry visual cylinder length=0.005 radius=0.0352
- link front_roll_link: geometry visual cylinder length=0.005 radius=0.0352
- link front_yaw_link: geometry visual cylinder length=0.005 radius=0.0352

File: xacro/barista_robot_model.urdf.xacro (robot description, xacro)
@@ -2,7 +2,8 @@
 <robot xmlns:xacro="http://www.ros.org/wiki/xacro" name="barista_robot">
   <!-- Conditional Argument -->
-  <xacro:property name="robot_name" value="$(arg robot_name)"/>
+  <xacro:property name="robot_name" default="barista"/>
   <xacro:arg name="robot_color" default="blue"/>
   <xacro:arg name="include_laser" default="true"/>
+  <xacro:property name="robot_name" value="$(arg robot_name)"/>
   <!-- Macro Includes -->
   <xacro:include filename="$(find barista_robot_description)/xacro/drive_wheel.xacro"/>

File: xacro/caster_wheel.xacro (robot description, xacro)
@@ -11,10 +11,4 @@
             <material name="$(arg robot_name)_black"/>
         </visual>
-        <collision>
-            <origin rpy="0 1.5707 1.5707" xyz="0 0 0"/>
-            <geometry>
-                <cylinder length="0.005" radius="0.0352"/>
-            </geometry>
-        </collision>
         <inertial>
             <mass value="0.01"/>
@@ -40,10 +34,4 @@
             <material name="$(arg robot_name)_black"/>
         </visual>
-        <collision>
-            <origin rpy="0 1.5707 1.5707" xyz="0 0 0"/>
-            <geometry>
-                <cylinder length="0.005" radius="0.0352"/>
-            </geometry>
-        </collision>
         <inertial>
             <mass value="0.01"/>
@@ -78,5 +66,5 @@
             <mass value="0.01"/>
             <origin rpy="0 0 0" xyz="0 0 0"/>
-            <inertia ixx="0.00000826" ixy="0" ixz="0" iyy="00.00000826" iyz="0" izz="0.00000826"/>
+            <inertia ixx="0.000004956" ixy="0" ixz="0" iyy="0.000004956" iyz="0" izz="0.000004956"/>
         </inertial>
     </link>
